Commit message: update name

File: unitree_description/a1_description/xacro/const.xacro (robot description, xacro)
@@ -29,6 +29,8 @@
     <xacro:property name="hip_offset" value="0.065"/>
     <!-- joint limits -->
-    <xacro:property name="damping" value="0"/>
-    <xacro:property name="friction" value="0"/>
+    <!-- <xacro:property name="damping" value="0"/> -->
+    <!-- <xacro:property name="friction" value="0"/> -->
+    <xacro:property name="damping" value="0.01"/>
+    <xacro:property name="friction" value="0.2"/>
     <xacro:property name="hip_max" value="46"/>
     <xacro:property name="hip_min" value="-46"/>
