Commit message: fix unitree hardware

File: unitree_description/a1_description/xacro/robot.xacro (robot description, xacro)
@@ -1,4 +1,6 @@
 <?xml version="1.0"?>
 <robot name="a1_description" xmlns:xacro="http://www.ros.org/wiki/xacro">
+    <xacro:arg name="use_gazebo" default="false"/>
+    <xacro:arg name="DEBUG" default="false"/>
     <xacro:include filename="$(find a1_description)/xacro/const.xacro"/>
     <xacro:include filename="$(find a1_description)/xacro/materials.xacro"/>
@@ -6,5 +8,5 @@
     <xacro:include filename="$(find a1_description)/xacro/stairs.xacro"/>
     <xacro:include filename="$(find a1_description)/xacro/gazebo.xacro"/>
-    <xacro:include filename="$(find a1_description)/xacro/ros2_control_interface.xacro"/>
+    <xacro:include filename="$(find a1_description)/xacro/ros2_control.xacro"/>
     <!-- <xacro:include filename="$(find a1_gazebo)/launch/stairs.urdf.xacro"/> -->
     <!-- <xacro:stairs stairs="15" xpos="0" ypos="0" zpos="0" /> -->
@@ -127,8 +129,8 @@
                 <plugin>unitree_hardware/UnitreeHardware</plugin>
             </hardware>
-            <xacro:leg_ros2_control_interface leg_name="FL"/>
-            <xacro:leg_ros2_control_interface leg_name="FR"/>
-            <xacro:leg_ros2_control_interface leg_name="RL"/>
-            <xacro:leg_ros2_control_interface leg_name="RR"/>
+            <xacro:leg_ros2_control leg_name="FL"/>
+            <xacro:leg_ros2_control leg_name="FR"/>
+            <xacro:leg_ros2_control leg_name="RL"/>
+            <xacro:leg_ros2_control leg_name="RR"/>
             <sensor name="IMU">
                 <state_interface name="orientation.x"/>
@@ -144,13 +146,17 @@
             </sensor>
             <sensor name="FL_foot_force_sensor">
+                <frame_id name="FL_foot"/>
                 <state_interface name="force.z"/>
             </sensor>
             <sensor name="FR_foot_force_sensor">
+                <frame_id name="FR_foot"/>
                 <state_interface name="force.z"/>
             </sensor>
             <sensor name="RL_foot_force_sensor">
+                <frame_id name="RL_foot"/>
                 <state_interface name="force.z"/>
             </sensor>
             <sensor name="RR_foot_force_sensor">
+                <frame_id name="RR_foot"/>
                 <state_interface name="force.z"/>
             </sensor>
@@ -163,8 +169,8 @@
                 <!-- <plugin>gazebo_ros2_control/GazeboSystem</plugin> -->
             </hardware>
-            <xacro:leg_ros2_control_interface leg_name="FL"/>
-            <xacro:leg_ros2_control_interface leg_name="FR"/>
-            <xacro:leg_ros2_control_interface leg_name="RL"/>
-            <xacro:leg_ros2_control_interface leg_name="RR"/>
+            <xacro:leg_ros2_control leg_name="FL"/>
+            <xacro:leg_ros2_control leg_name="FR"/>
+            <xacro:leg_ros2_control leg_name="RL"/>
+            <xacro:leg_ros2_control leg_name="RR"/>
             <sensor name="imu_sensor">
                 <frame_id name="imu_link"/>

File: unitree_description/a1_description/xacro/ros2_control.xacro (robot description, xacro)
@@ -1,5 +1,5 @@
 <?xml version="1.0"?>
 <robot xmlns:xacro="http://www.ros.org/wiki/xacro">
-    <xacro:macro name="leg_ros2_control_interface" params="leg_name">
+    <xacro:macro name="leg_ros2_control" params="leg_name">
         <joint name="${leg_name}_hip_joint">
             <command_interface name="position">
